File: Electrical-flight controller/Version-1/Version-1.kicad_sch (KiCad schematic)
At the start: 4 parts, among them U1 MPU-6050, U2 ATmega328P-A, U3 BMP280, U4 LM1117DT-ADJ

Commit message: Started ESP32
Parts:
- removed U1: MPU-6050, Sensor_Motion:InvenSense_QFN-24_4x4mm_P0.5mm, symbol Sensor_Motion:MPU-6050
- removed U2: ATmega328P-A, Package_QFP:TQFP-32_7x7mm_P0.8mm, symbol MCU_Microchip_ATmega:ATmega328P-A
- removed U3: BMP280, Package_LGA:Bosch_LGA-8_2x2.5mm_P0.65mm_ClockwisePinNumbering, symbol Sensor_Pressure:BMP280
- removed U4: LM1117DT-ADJ, Package_TO_SOT_SMD:TO-252-3_TabPin2, symbol Regulator_Linear:LM1117DT-ADJ
- added U1: ESP32-WROOM-32, RF_Module:ESP32-WROOM-32, symbol RF_Module:ESP32-WROOM-32
Connections:
- new net: U1.1 (GND), U1.15 (GND), U1.38 (GND), U1.39 (GND)

Commit message: 2nd update
Parts:
- added U2: W25Q32JVZP, Package_SON:WSON-8-1EP_6x5mm_P1.27mm_EP3.4x4.3mm, symbol Memory_Flash:W25Q32JVZP
- added Y1: Crystal_GND24, symbol Device:Crystal_GND24
Changed lines of the file:
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@@
 	(paper "A4")
+	(symbol
+		(lib_id "Device:Crystal_GND24")
+		(at 170.18 78.74 0)
+		(unit 1)
+		(exclude_from_sim no)
+		(in_bom yes)
+		(on_board yes)
+		(dnp no)
+		(fields_autoplaced yes)
+		(property "Reference" "Y1"
+			(at 181.61 72.3198 0)
+			(effects
+				(font
+					(size 1.27 1.27)
+				)
+			)
+		)
+		(property "Value" "Crystal_GND24"
+			(at 181.61 74.8598 0)
+			(effects
+				(font
+					(size 1.27 1.27)
+				)
+			)
+		)
+		(property "Footprint" ""
+			(at 170.18 78.74 0)
+			(effects
+				(font
+					(size 1.27 1.27)
+				)
+				(hide yes)
+			)
+		)
+		(property "Datasheet" "~"
+			(at 170.18 78.74 0)
+			(effects
+				(font
+					(size 1.27 1.27)
+				)
+				(hide yes)
+			)
+		)
+		(property "Description" "Four pin crystal, GND on pins 2 and 4"
+			(at 170.18 78.74 0)
+			(effects
+				(font
+					(size 1.27 1.27)
+				)
+				(hide yes)
+			)
+		)
+		(pin "1"
+		)
+		(pin "2"
+		)
+		(pin "3"
+		)
+		(pin "4"
+		)
+		(instances
+			(project ""
+				(path "/b01821f6-bde1-4035-92df-fac2c021cb26"
+					(reference "Y1")
+					(unit 1)
+				)
+			)
+		)
+	)
+	(symbol
+		(lib_id "Memory_Flash:W25Q32JVZP")
+		(at 69.85 48.26 0)
+		(unit 1)
+		(exclude_from_sim no)
+		(in_bom yes)
+		(on_board yes)
+		(dnp no)
+		(fields_autoplaced yes)
+		(property "Reference" "U2"
+			(at 81.28 46.9899 0)
+			(effects
+				(font
+					(size 1.27 1.27)
+				)
+				(justify left)
+			)
+		)
+		(property "Value" "W25Q32JVZP"
+			(at 81.28 49.5299 0)
+			(effects
+				(font
+					(size 1.27 1.27)
+				)
+				(justify left)
+			)
+		)
+		(property "Footprint" "Package_SON:WSON-8-1EP_6x5mm_P1.27mm_EP3.4x4.3mm"
+			(at 69.85 48.26 0)
+			(effects
+				(font
+					(size 1.27 1.27)
+				)
+				(hide yes)
+			)
+		)
+		(property "Datasheet" "http://www.winbond.com/resource-files/w25q32jv%20revg%2003272018%20plus.pdf"
+			(at 69.85 50.8 0)
+			(effects
+				(font
+					(size 1.27 1.27)
+				)
+				(hide yes)
+			)
+		)
+		(property "Description" "32Mbit / 4MiB Serial Flash Memory, Standard/Dual/Quad SPI, 2.7-3.6V, WSON-8"
+			(at 69.85 48.26 0)
+			(effects
+				(font
+					(size 1.27 1.27)
+				)
+				(hide yes)
+			)
+		)
+		(pin "5"
+		)
+		(pin "7"
+		)
+		(pin "2"
+		)
+		(pin "9"
+		)
+		(pin "1"
+		)
+		(pin "6"
+		)
+		(pin "3"
+		)
+		(pin "8"
+		)
+		(pin "4"
+		)
+		(instances
+			(project ""
+				(path "/b01821f6-bde1-4035-92df-fac2c021cb26"
+					(reference "U2")
+					(unit 1)
+				)
+			)
+		)
+	)
 	(symbol
 		(lib_id "RF_Module:ESP32-WROOM-32")

Commit message: power circuit
Parts:
- added C1: 10u, symbol Device:C
- added C2: 0u1, symbol Device:C
- added D2, D3, D4: LESD5D5.0CT1G, symbol Device:D_TVS
- added D5: 1N5819, Diode_THT:D_DO-41_SOD81_P10.16mm_Horizontal, symbol Diode:1N5819
- added D6: LED, LED_SMD:LED_0201_0603Metric, symbol Device:LED
- added J1: USB_B_Micro, symbol Connector:USB_B_Micro
- added R1, R2, R3, R5, R6, R7: 0, symbol Device:R
- added R4: 330, Resistor_SMD:R_0402_1005Metric, symbol Device:R
- added U4: CP2102N-Axx-xQFN28, Package_DFN_QFN:QFN-28-1EP_5x5mm_P0.5mm_EP3.35x3.35mm, symbol Interface_USB:CP2102N-Axx-xQFN28
Connections:
- new net: D6.2 (A), R4.1
- new net: D3.1 (A1), J1.3 (D+), R1.1
- new net: D4.1 (A1), J1.2 (D-), R2.1
- new net: D2.1 (A1), D5.2 (A), J1.1 (VBUS), R4.2
- new net 5v: C1.1, C2.1, D5.1 (K), U4.8 (VBUS)
- new net CTS: R7.2
- new net GND: C1.2, C2.2, D2.2 (A2), D3.2 (A2), D4.2 (A2), D6.1 (K), J1.5 (GND), U4.29 (GND), U4.3 (GND)
- new net IO13: R6.1
- new net IO15: R7.1
- new net RTS: R6.2
- new net RXD: R5.2, U4.25 (RXD)
- new net RXD0: R5.1
- new net TXD: R3.2, U4.26 (TXD)
- new net TXD0: R3.1
- new net USB_DN: R2.2
- new net USB_DP: R1.2, U4.4 (D+), U4.5 (D-)
- no-connect marks 0 -> 18
Other:
- moved on the sheet: U1, U2, Y1

Commit message: Pwoer supply
Parts:
- removed D6: LED, LED_SMD:LED_0201_0603Metric, symbol Device:LED
- removed Y1: Crystal_GND24, symbol Device:Crystal_GND24
- added C3, C4: 10uF, symbol Device:C
- added C5: 0.1uF, symbol Device:C
- added D1: LED, symbol Device:LED
- added Q1, Q2: S8050, Package_TO_SOT_THT:TO-92_Inline, symbol Transistor_BJT:S8050
- added R8, R9: 10K, symbol Device:R
- added U3: 74LS04, symbol 74xx:74LS04
- added U5: AMS1117, Package_TO_SOT_SMD:SOT-223-3_TabPin2, symbol Regulator_Linear:AMS1117
- added Y2: ASE-xxxMHz, Oscillator:Oscillator_SMD_Abracon_ASE-4Pin_3.2x2.5mm, symbol Oscillator:ASE-xxxMHz
- C1: value 10u -> 10uF
- C2: value 0u1 -> 0.1uF
- R4: value 330 -> 2K; footprint Resistor_SMD:R_0402_1005Metric -> (none)
Connections:
- net 5v: now also R4.1, C3.1, U3.14 (VCC), U5.3 (VI)
- net CTS: now also U3.4
- net GND: now also C3.2, C4.2, C5.2, D1.1 (K), U3.7 (GND), U5.1 (ADJ)
- net RTS: now also Q1.1 (E), R9.1, U3.2
- net at D2.1 (A1), D5.2 (A), J1.1 (VBUS): no longer R4.2
- net at U4.23 (~{CTS}): now also U3.3
- net at U4.24 (~{RTS}): now also U3.1
- net at U4.28 (~{DTR}): now also U3.5
- net 3.3v: now reaches U4.6 (VDD)
- net 3.3v: now also U1.2 (VDD), U4.7 (VREGIN), C4.1, C5.1, U5.2 (VO)
- new net: Q2.2 (B), R9.2
- new net: D1.2 (A), R4.2
- new net: Q1.2 (B), R8.2
- new net DTR: Q2.1 (E), R8.1, U3.6
- new net EN: Q1.3 (C)
- new net IO0: Q2.3 (C)
Other:
- note added: "Power regulator"
- moved on the sheet: U1, U2

Commit message: flash chip, reset switches , mc etc
Parts:
- removed U2: W25Q32JVZP, Package_SON:WSON-8-1EP_6x5mm_P1.27mm_EP3.4x4.3mm, symbol Memory_Flash:W25Q32JVZP
- removed Y2: ASE-xxxMHz, Oscillator:Oscillator_SMD_Abracon_ASE-4Pin_3.2x2.5mm, symbol Oscillator:ASE-xxxMHz
- added BZ1: Buzzer, Buzzer_Beeper:MagneticBuzzer_Kingstate_KCG0601, symbol Device:Buzzer
- added C10, C11: 22p, Capacitor_SMD:C_0201_0603Metric, symbol Device:C
- added C6: 0.1uF, symbol Device:C
- added C7, C8: 1nF, symbol Device:C
- added C9: 0u1, Capacitor_SMD:C_0201_0603Metric, symbol Device:C
- added D6: ESD3.3V88D-C, symbol Device:D_TVS
- added J2, J3: Conn_01x02_Pin, symbol Connector:Conn_01x02_Pin
- added JP3, JP4: Jumper_2_Small_Open, Jumper:SolderJumper-2_P1.3mm_Open_Pad1.0x1.5mm, symbol Jumper:Jumper_2_Small_Open
- added Q4: BSS138, Package_TO_SOT_SMD:SOT-23, symbol Transistor_FET:BSS138
- added R10, R11, R12, R13: 100R, symbol Device:R
- added R14: 10K, symbol Device:R
- added R15, R16: 47R, symbol Device:R
- added R17, R18, R34: 2k2, Resistor_SMD:R_0402_1005Metric, symbol Device:R
- added R19, R20: 4k7, Resistor_SMD:R_0402_1005Metric, symbol Device:R
- added R21: 10k, Resistor_SMD:R_0402_1005Metric, symbol Device:R
- added SW1, SW2: SW_MEC_5G, symbol Switch:SW_MEC_5G
- added U2: W25Q128JVE, Package_SON:WSON-8-1EP_8x6mm_P1.27mm_EP3.4x4.3mm, symbol Memory_Flash:W25Q128JVE
- added U6: BMP390L, barometer:XDCR_BMP390L.kicad_mod, symbol BMP390L:BMP390L
- added U8: BNO055, Package_LGA:LGA-28_5.2x3.8mm_P0.5mm, symbol Sensor_Motion:BNO055
- added Y1: Crystal, Crystal:Crystal_C26-LF_D2.1mm_L6.5mm_Vertical, symbol Device:Crystal
Connections:
- net 3.3v: now also D6.1 (A1), R14.1, U2.8 (VCC)
- net EN: now also U1.3 (EN), C6.1, R14.2, R16.1
- net GND: now also U1.1 (GND), U1.15 (GND), U1.38 (GND), U1.39 (GND), C10.2, C11.2, C6.2, C7.1, C8.1, C9.2, D6.2 (A2), JP4.2 (B), Q4.2 (S), R34.2, SW1.1 (A), SW1.2 (A), SW2.1 (A), SW2.2 (A), U6.3 (VSS/GND), U6.8 (VSS/GND), U6.9 (VSS/GND), U8.2 (GND), U8.25 (GNDIO)
- net IO0: now also U1.25 (IO0), R15.1
- net RXD0: now also U1.34 (RXD0/IO3)
- net TXD0: now also U1.35 (TXD0/IO1)
- net at U1.13 (IO14): now also R10.1
- net at U1.14 (IO12): now also R11.1
- net at U1.16 (IO13): now also R12.1
- net at U1.23 (IO15): now also R13.1
- net BUZZER: now reaches U1.24 (IO2)
- net BUZZER: now also Q4.1 (G), R34.1
- new net: C10.1, U8.26 (XOUT32), Y1.2
- new net: C9.1, U8.9 (CAP)
- new net: J2.1 (Pin_1), R11.2
- new net: J2.2 (Pin_2), R10.2
- new net: BZ1.2 (-), Q4.3 (D)
- new net: J3.1 (Pin_1), R13.2
- new net: R21.1, U8.11 (~{RESET})
- new net: J3.2 (Pin_2), R12.2
- new net: C8.2, R16.2, SW2.3 (B), SW2.4 (B)
- new net: C11.1, U8.27 (XIN32), Y1.1
- new net: C7.2, R15.2, SW1.3 (B), SW1.4 (B)
- new net: JP3.1 (A), JP4.1 (A), U6.5 (SDO/DNC/SA0)
- new net +3.3V: BZ1.1 (+), JP3.2 (B), R17.1, R18.1, R19.1, R20.1, R21.2, U6.1 (VDDIO), U6.10 (VDD), U6.6 (~{CS}), U8.28 (VDDIO), U8.3 (VDD)
- new net SCL: R18.2, R20.2, U6.2 (SCK/SCL), U8.17 (COM3)
- new net SDA: R17.2, R19.2, U6.4 (SDI/SDO/SDA), U8.18 (COM2)
- no-connect marks 18 -> 26

Commit message: 123
Parts:
- removed JP3, JP4: Jumper_2_Small_Open, Jumper:SolderJumper-2_P1.3mm_Open_Pad1.0x1.5mm, symbol Jumper:Jumper_2_Small_Open
Connections:
- net SCL is gone; now on net SCK: R18.2, R20.2, U6.2 (SCK/SCL), U8.17 (COM3)
- net SDA is gone; now on net SENSOR: R17.2, R19.2, U6.4 (SDI/SDO/SDA), U8.18 (COM2)
- net +3.3V: no longer R17.1, R18.1, R19.1, R20.1, R21.2, U6.1 (VDDIO), U6.10 (VDD), U6.6 (~{CS}), U8.28 (VDDIO), U8.3 (VDD)
- net 3.3v: now also R17.1, R18.1, R19.1, R20.1, R21.2, U6.1 (VDDIO), U6.10 (VDD), U6.6 (~{CS}), U8.28 (VDDIO), U8.3 (VDD)
- net GND: now also U2.4 (GND)
- net CS: now reaches U2.1 (~{CS})
- net CS: now also U1.26 (IO4)
- net DO: now reaches U2.2 (DO/IO_{1})
- net DO: now also U1.27 (IO16)
- net DI: now reaches U2.5 (DI/IO_{0})
- net DI: now also U1.29 (IO5)
- net SCK: now reaches U2.6 (CLK)
- net SCK: now also U1.20 (SCK/CLK)
- net EP: now reaches U2.9 (EP)
- net EP: now also U1.28 (IO17)
- net SENSOR: now reaches U1.7 (IO35)
- no-connect marks 26 -> 29
Other:
- moved on the sheet: U2
