File: Electrical-flight controller/Version-1/Version-1.kicad_sch (KiCad schematic)
At the start: 56 parts, among them J1 USB_B_Micro, J2 Conn_01x02_Pin, J3 Conn_01x02_Pin, Q1 S8050, Q2 S8050, Q4 BSS138, SW1 SW_MEC_5G, SW2 SW_MEC_5G, U1 ESP32-WROOM-32, U2 W25Q128JVE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

Commit message: light earlier changes
Connections:
- net SCK: no longer U1.20 (SCK/CLK)
Other:
- moved on the sheet: R17, R18, R21, U8

Commit message: some changes in wiring of IMU and flash and bmp -> not fully done:(
Parts:
- removed C10, C11: 22p, Capacitor_SMD:C_0201_0603Metric, symbol Device:C
- removed C9: 0u1, Capacitor_SMD:C_0201_0603Metric, symbol Device:C
- removed R17, R18: 2k2, Resistor_SMD:R_0402_1005Metric, symbol Device:R
- removed U8: BNO055, Package_LGA:LGA-28_5.2x3.8mm_P0.5mm, symbol Sensor_Motion:BNO055
- removed Y1: Crystal, Crystal:Crystal_C26-LF_D2.1mm_L6.5mm_Vertical, symbol Device:Crystal
- added R22: 4k7, Resistor_SMD:R_0402_1005Metric, symbol Device:R
- added U7: ICM-20948, Sensor_Motion:InvenSense_QFN-24_3x3mm_P0.4mm, symbol Sensor_Motion:ICM-20948
- R21: value 10k -> 4k7
Connections:
- net 3.3v: now also R21.1, U6.5 (SDO/DNC/SA0), R22.1, U7.13 (VDD), U7.22 (~{CS}), U7.8 (VDDIO), U7.9 (SDO/AD0); no longer R21.2
- net DI: no longer U1.29 (IO5)
- net DO: no longer U1.27 (IO16)
- net EP: no longer U1.28 (IO17)
- net GND: now also U7.18 (GND), U7.20 (GND)
- net SCK: no longer R20.2, U6.2 (SCK/SCL)
- net SENSOR: no longer R19.2, U6.4 (SDI/SDO/SDA)
- new net: R21.2, U7.23 (SCL/SCLK)
- new net: R19.2, U6.4 (SDI/SDO/SDA)
- new net: R22.2, U7.24 (SDA/SDI)
- new net: R20.2, U6.2 (SCK/SCL)
- no-connect marks 29 -> 26

Commit message: main schemtic done!!
Parts:
- removed J2, J3: Conn_01x02_Pin, symbol Connector:Conn_01x02_Pin
- removed R10, R11, R12, R13: 100R, symbol Device:R
- added J2: Conn_01x08_Socket, symbol Connector:Conn_01x08_Socket
- added R23, R24: 4k7, Resistor_SMD:R_0402_1005Metric, symbol Device:R
Connections:
- net SENSOR is gone; now on net I2C-D: U1.7 (IO35)
- net +3.3V: now also J2.3 (Pin_3)
- net 3.3v: now also R23.1, R24.1
- net BUZZER: now also U1.33 (IO21); no longer U1.24 (IO2)
- net CS: now also U1.9 (IO33); no longer U1.26 (IO4)
- net DI: now also U1.13 (IO14)
- net DO: now also U1.27 (IO16)
- net GND: now also J2.4 (Pin_4), J2.8 (Pin_8)
- net SCK: now also U1.16 (IO13), U1.30 (IO18), J2.5 (Pin_5)
- net I2C-CL: now reaches R21.2, U7.23 (SCL/SCLK)
- net I2C-CL: now also R20.2, U1.28 (IO17), U6.2 (SCK/SCL), J2.1 (Pin_1), R24.2
- net I2C-D: now reaches R19.2, U6.4 (SDI/SDO/SDA)
- net I2C-D: now also R22.2, U7.24 (SDA/SDI), J2.2 (Pin_2), R23.2
- net esc_1: now reaches U1.10 (IO25)
- net esc_2: now reaches U1.11 (IO26)
- net esc_3: now reaches U1.12 (IO27)
- net MISO: now reaches U1.31 (IO19)
- net MISO: now also J2.6 (Pin_6)
- net MOSI: now reaches U1.37 (IO23)
- net MOSI: now also J2.7 (Pin_7)
- net esc_4: now reaches U1.8 (IO32)
- no-connect marks 26 -> 32
Other:
- note added: "0x30"
- note added: "CAM"
- note added: "Flash chip"
- note added: "Gyroscope"
- note added: "LIPO"
- note added: "Microcontroller"
- note added: "Motor"
- note added: "Pressure sensor"
- moved on the sheet: R22, U2
